File: 2018 Q1/EAGLE Files/OPEnSampler r2/March22.sch (EAGLE design)
At the start: 30 parts, among them IC1 TPIC6B596N, IC2 TPIC6B596N, IC3 TPIC6B596N, IC4 TPIC6B596N

Commit message: added sch file
Parts:
- added R_DOWN, R_UP: (no value), adafruit:R-US_0204/7
- added STATE_JUMPER: (no value), jumper:JP2E
- added U1: MMPQ2222A, MMPQ2222A:MMPQ2222A
Connections:
- new net N$15: R_DOWN.1, U1.E, U1.E_4
- new net N$9: R_UP.1, STATE_JUMPER.2, U$2.STATE
- new net POW_OFF: MS1.GPIO11, U1.B_3
- net 12V: now also R_UP.2, U1.E_3
- net 5V: now also U1.B
- net GND: now also U1.C_2, U1.C_4
- net REG_EN: now also R_DOWN.2, STATE_JUMPER.3, U1.C_6; no longer U$2.STATE
- net RTC_SQW: now also U1.B_4
Other:
- note added: "POWER CIRCUIT"
Changed lines of the file:
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@@
 <?xml version="1.0" encoding="utf-8"?>
 <!DOCTYPE eagle SYSTEM "eagle.dtd">
-<eagle version="8.7.0">
+<eagle version="8.6.3">
 <drawing>
 <settings>
-<setting alwaysvectorfont="yes"/>
+<setting alwaysvectorfont="no"/>
 <setting verticaltext="up"/>
 </settings>
@@
 <layer number="132" name="bAdjust" color="7" fill="1" visible="no" active="yes"/>
 <layer number="144" name="Drill_legend" color="7" fill="1" visible="no" active="yes"/>
-<layer number="150" name="Notes" color="7" fill="1" visible="no" active="yes"/>
+<layer number="150" name="Notes" color="7" fill="1" visible="yes" active="yes"/>
 <layer number="151" name="HeatSink" color="7" fill="1" visible="no" active="yes"/>
 <layer number="152" name="_bDocu" color="7" fill="1" visible="no" active="yes"/>
@@
 <part name="POWER" library="adafruit" deviceset="2.1MMJACK" device="SMT"/>
 <part name="GND8" library="SparkFun-PowerSymbols" deviceset="GND" device=""/>
+<part name="U1" library="MMPQ2222A" deviceset="MMPQ2222A" device=""/>
+<part name="R_DOWN" library="adafruit" deviceset="R-US_" device="0204/7"/>
+<part name="GND9" library="supply1" library_urn="urn:adsk.eagle:library:371" deviceset="GND" device=""/>
+<part name="STATE_JUMPER" library="jumper" library_urn="urn:adsk.eagle:library:252" deviceset="JP2E" device="" package3d_urn="urn:adsk.eagle:package:15452/1"/>
+<part name="R_UP" library="adafruit" deviceset="R-US_" device="0204/7"/>
 </parts>
 <sheets>
 <sheet>
 <plain>
+<wire x1="187.96" y1="-33.02" x2="187.96" y2="63.5" width="0.1524" layer="150"/>
+<wire x1="187.96" y1="63.5" x2="281.94" y2="63.5" width="0.1524" layer="150"/>
+<wire x1="281.94" y1="63.5" x2="281.94" y2="-33.02" width="0.1524" layer="150"/>
+<wire x1="281.94" y1="-33.02" x2="187.96" y2="-33.02" width="0.1524" layer="150"/>
+<text x="190.5" y="55.88" size="5.08" layer="150">POWER CIRCUIT</text>
 </plain>
 <instances>
@@
 <instance part="POWER" gate="G$1" x="198.12" y="50.8" rot="R270"/>
 <instance part="GND8" gate="1" x="195.58" y="20.32"/>
+<instance part="U1" gate="A" x="210.82" y="-5.08"/>
+<instance part="R_DOWN" gate="G$1" x="259.08" y="2.54" rot="R90"/>
+<instance part="GND9" gate="1" x="205.74" y="-7.62"/>
+<instance part="STATE_JUMPER" gate="1" x="231.14" y="15.24" rot="R270"/>
+<instance part="R_UP" gate="G$1" x="220.98" y="15.24" rot="R180"/>
 </instances>
 <busses>
@@
 <junction x="195.58" y="22.86"/>
 <pinref part="GND8" gate="1" pin="GND"/>
+</segment>
+<segment>
+<pinref part="U1" gate="A" pin="C_2"/>
+<wire x1="213.36" y1="-5.08" x2="210.82" y2="-5.08" width="0.1524" layer="91"/>
+<pinref part="GND9" gate="1" pin="GND"/>
+<wire x1="210.82" y1="-5.08" x2="205.74" y2="-5.08" width="0.1524" layer="91"/>
+<wire x1="210.82" y1="-5.08" x2="210.82" y2="-10.16" width="0.1524" layer="91"/>
+<pinref part="U1" gate="A" pin="C_4"/>
+<wire x1="210.82" y1="-10.16" x2="213.36" y2="-10.16" width="0.1524" layer="91"/>
 </segment>
 </net>
@@
 <pinref part="MS1" gate="G$1" pin="GPIOA0"/>
 <wire x1="15.24" y1="33.02" x2="43.18" y2="33.02" width="0.1524" layer="91"/>
+</segment>
+<segment>
+<pinref part="U1" gate="A" pin="B_4"/>
+<label x="254" y="-12.7" size="1.27" layer="95"/>
+<wire x1="254" y1="-12.7" x2="261.62" y2="-12.7" width="0.1524" layer="91"/>
 </segment>
 </net>
@@
 </segment>
 <segment>
+<pinref part="U1" gate="A" pin="B"/>
+<label x="254" y="-7.62" size="1.27" layer="95"/>
+<wire x1="254" y1="-7.62" x2="276.86" y2="-7.62" width="0.1524" layer="91"/>
 <pinref part="C12" gate="G$1" pin="+"/>
 <wire x1="261.62" y1="38.1" x2="269.24" y2="38.1" width="0.1524" layer="91"/>
@@
 <wire x1="269.24" y1="45.72" x2="238.76" y2="45.72" width="0.1524" layer="91"/>
 <pinref part="L1" gate="G$1" pin="B"/>
-<wire x1="269.24" y1="45.72" x2="279.4" y2="45.72" width="0.1524" layer="91"/>
+<wire x1="269.24" y1="45.72" x2="276.86" y2="45.72" width="0.1524" layer="91"/>
 <junction x="269.24" y="45.72"/>
 <label x="274.32" y="45.72" size="1.778" layer="95"/>
+<wire x1="276.86" y1="-7.62" x2="276.86" y2="45.72" width="0.1524" layer="91"/>
+<junction x="276.86" y="45.72"/>
 </segment>
 </net>
@@
 <wire x1="213.36" y1="45.72" x2="205.74" y2="45.72" width="0.1524" layer="91"/>
 <junction x="205.74" y="45.72"/>
+<pinref part="R_UP" gate="G$1" pin="2"/>
+<wire x1="215.9" y1="15.24" x2="200.66" y2="15.24" width="0.1524" layer="91"/>
+<wire x1="200.66" y1="15.24" x2="200.66" y2="45.72" width="0.1524" layer="91"/>
+<junction x="200.66" y="45.72"/>
 </segment>
 <segment>
@@
 <label x="152.4" y="2.54" size="1.27" layer="95"/>
 </segment>
+<segment>
+<pinref part="U1" gate="A" pin="E_3"/>
+<wire x1="254" y1="-15.24" x2="261.62" y2="-15.24" width="0.1524" layer="91"/>
+<label x="259.08" y="-15.24" size="1.27" layer="95"/>
+</segment>
 </net>
 <net name="REG_EN" class="0">
 <segment>
+<label x="225.806" y="23.622" size="1.778" layer="95" rot="R90"/>
+<wire x1="259.08" y1="7.62" x2="228.6" y2="7.62" width="0.1524" layer="91"/>
+<pinref part="R_DOWN" gate="G$1" pin="2"/>
+<pinref part="U1" gate="A" pin="C_6"/>
+<wire x1="228.6" y1="7.62" x2="200.66" y2="7.62" width="0.1524" layer="91"/>
+<wire x1="213.36" y1="-15.24" x2="200.66" y2="-15.24" width="0.1524" layer="91"/>
+<wire x1="200.66" y1="-15.24" x2="200.66" y2="7.62" width="0.1524" layer="91"/>
+<pinref part="STATE_JUMPER" gate="1" pin="3"/>
+<wire x1="228.6" y1="7.62" x2="228.6" y2="12.7" width="0.1524" layer="91"/>
+<junction x="228.6" y="7.62"/>
+</segment>
+</net>
+<net name="POW_OFF" class="0">
+<segment>
+<pinref part="U1" gate="A" pin="B_3"/>
+<wire x1="254" y1="-17.78" x2="261.62" y2="-17.78" width="0.1524" layer="91"/>
+<label x="254" y="-17.78" size="1.27" layer="95"/>
+</segment>
+<segment>
+<pinref part="MS1" gate="G$1" pin="GPIO11"/>
+<wire x1="86.36" y1="20.32" x2="91.44" y2="20.32" width="0.1524" layer="91"/>
+<label x="88.9" y="20.32" size="1.27" layer="95"/>
+</segment>
+</net>
+<net name="N$15" class="0">
+<segment>
+<pinref part="R_DOWN" gate="G$1" pin="1"/>
+<pinref part="U1" gate="A" pin="E_4"/>
+<wire x1="254" y1="-10.16" x2="259.08" y2="-10.16" width="0.1524" layer="91"/>
+<wire x1="259.08" y1="-10.16" x2="259.08" y2="-5.08" width="0.1524" layer="91"/>
+<pinref part="U1" gate="A" pin="E"/>
+<wire x1="259.08" y1="-5.08" x2="259.08" y2="-2.54" width="0.1524" layer="91"/>
+<wire x1="254" y1="-5.08" x2="259.08" y2="-5.08" width="0.1524" layer="91"/>
+<junction x="259.08" y="-5.08"/>
+</segment>
+</net>
+<net name="N$9" class="0">
+<segment>
+<pinref part="STATE_JUMPER" gate="1" pin="2"/>
+<wire x1="228.6" y1="15.24" x2="226.06" y2="15.24" width="0.1524" layer="91"/>
 <pinref part="U$2" gate="G$1" pin="STATE"/>
-<wire x1="226.06" y1="33.02" x2="226.06" y2="30.48" width="0.1524" layer="91"/>
-<wire x1="226.06" y1="30.48" x2="233.68" y2="30.48" width="0.1524" layer="91"/>
-<label x="226.822" y="30.734" size="1.778" layer="95"/>
+<wire x1="226.06" y1="15.24" x2="226.06" y2="33.02" width="0.1524" layer="91"/>
+<pinref part="R_UP" gate="G$1" pin="1"/>
+<junction x="226.06" y="15.24"/>
 </segment>
 </net>
@@
 </schematic>
 </drawing>
+<compatibility>
+<note version="8.2" severity="warning">
+Since Version 8.2, EAGLE supports online libraries. The ids
+of those online libraries will not be understood (or retained)
+with this version.
+</note>
+<note version="8.3" severity="warning">
+Since Version 8.3, EAGLE supports URNs for individual library
+assets (packages, symbols, and devices). The URNs of those assets
+will not be understood (or retained) with this version.
+</note>
+<note version="8.3" severity="warning">
+Since Version 8.3, EAGLE supports the association of 3D packages
+with devices in libraries, schematics, and board files. Those 3D
+packages will not be understood (or retained) with this version.
+</note>
+</compatibility>
 </eagle>
